Commit message: simple robot demo

File: my_robot_pkg/urdf/my_mobile_robot_simple.xacro (robot description, xacro)
@@ -24,5 +24,5 @@
     </visual>
   </link>
-<link name="right_wheel">
+  <link name="right_wheel">
     <visual name="right_wheel_visual">
       <origin xyz="0 0 0" rpy="0 1.5707 1.5707"/>
